Commit message: added thw world file

File: description/lidar.xacro (robot description, xacro)
@@ -4,5 +4,5 @@
         <parent link="chassis"/>
         <child link="laser_frame"/>
-        <origin xyz="0.1 0 0.175" rpy="0 0 0"/>
+        <origin xyz="0.1 0 0.125" rpy="0 0 0"/>
     </joint>
     <link name="laser_frame">

File: description/robot_core.xacro (robot description, xacro)
@@ -100,5 +100,5 @@
         <parent link="chassis"/>
         <child link="caster_wheel"/>
-        <origin xyz="0.17 0 0"/>
+        <origin xyz="0.16 0 0"/>
     </joint>
     <link name="caster_wheel">
@@ -114,5 +114,5 @@
             </geometry>
         </collision>
-        <xacro:inertial_sphere mass="0.1" radius="0.05">
+        <xacro:inertial_sphere mass="0.9" radius="0.05">
             <origin xyz="0 0 0" rpy="0 0 0"/>
         </xacro:inertial_sphere>

Commit message: new fixes done

File: description/lidar.xacro (robot description, xacro)
@@ -26,5 +26,5 @@
         <sensor name="laser" type="ray">
             <pose> 0 0 0 0 0 0 </pose>
-            <visualize>true</visualize>
+            <visualize>false</visualize>
             <update_rate>10</update_rate>
             <ray>

File: description/robot_core.xacro (robot description, xacro)
@@ -17,4 +17,11 @@
     <link name="base_link">
     </link>
+    <!-- BASE_FOOTPRINT LINK -->
+    <joint name="base_footprint_joint" type="fixed">
+        <parent link="base_link"/>
+        <child link="base_footprint"/>
+        <origin xyz="0 0 0" rpy="0 0 0"/>
+    </joint>
+    <link name="base_footprint"></link>
     <!-- CHASSIS LINK -->
     <joint name="chassis_joint" type="fixed">

Commit message: new

File: description/lidar.xacro (robot description, xacro)
@@ -4,5 +4,5 @@
         <parent link="chassis"/>
         <child link="laser_frame"/>
-        <origin xyz="0.122 0 0.212" rpy="0 0 0"/>
+        <origin xyz="-0.122 0 0.109" rpy="0 0 0"/>
     </joint>
     <link name="laser_frame">

Commit message: mew

File: description/lidar.xacro (robot description, xacro)
@@ -4,5 +4,5 @@
         <parent link="chassis"/>
         <child link="laser_frame"/>
-        <origin xyz="-0.122 0 0.109" rpy="0 0 0"/>
+        <origin xyz="0.122 0 0.109" rpy="0 0 0"/>
     </joint>
     <link name="laser_frame">

Commit message: mew

File: description/lidar.xacro (robot description, xacro)
@@ -4,5 +4,5 @@
         <parent link="chassis"/>
         <child link="laser_frame"/>
-        <origin xyz="0.122 0 0.109" rpy="0 0 0"/>
+        <origin xyz="0.08 0 0.109" rpy="0 0 0"/>
     </joint>
     <link name="laser_frame">

Commit message: today

File: description/lidar.xacro (robot description, xacro)
@@ -4,5 +4,5 @@
         <parent link="chassis"/>
         <child link="laser_frame"/>
-        <origin xyz="0.05625 0 0.109" rpy="0 0 0"/>
+        <origin xyz="0.05625 0 0.13" rpy="0 0 0"/>
     </joint>
     <link name="laser_frame">
@@ -32,6 +32,6 @@
                     <horizontal>
                         <samples>360</samples>
-                        <min_angle>-1.57</min_angle>
-                        <max_angle>1.57</max_angle>
+                        <min_angle>-3.14</min_angle>
+                        <max_angle>3.14</max_angle>
                     </horizontal>
                 </scan>

File: description/robot_core.xacro (robot description, xacro)
@@ -70,5 +70,5 @@
         <parent link="base_link"/>
         <child link="left_wheel"/>
-        <origin xyz="0 0.1265 0" rpy="-${pi/2} 0 0" />
+        <origin xyz="0 0.15 0" rpy="-${pi/2} 0 0" />
         <axis xyz="0 0 1"/>
     </joint>
@@ -96,5 +96,5 @@
         <parent link="base_link"/>
         <child link="right_wheel"/>
-        <origin xyz="0 -0.1265 0" rpy="${pi/2} 0 0" />
+        <origin xyz="0 -0.15 0" rpy="${pi/2} 0 0" />
         <axis xyz="0 0 -1"/>
     </joint>
